Commit message: added loading in gazebo and pid

File: robotiq_3f_gazebo/robots/robotiq_3f_gripper.urdf.gazebo.xacro (robot description, xacro)
@@ -4,9 +4,9 @@
   <xacro:include filename="$(find robotiq_3f_gazebo)/robots/robotiq_3f_gripper.gazebo.xacro"/>
   <xacro:include filename="$(find robotiq_3f_gazebo)/robots/robotiq_3f_gripper.gazebo.macro.xacro"/>
-  <link name="world" />
+  <!-- <link name="world" />
   <joint name="joint_w" type="fixed">
     <parent link="world"/>
     <child link="palm"/>
     <origin xyz="0 0 0.054" rpy="1.57 0 0"/>
-  </joint>
+  </joint> -->
 </robot>
